Commit message: TCP control of car

File: src/assets/chevy.urdf (robot description, URDF)
Before this commit: robot Chevy, 8 links, 7 joints
Links:
- added link front_axle, mass 8.0; visual cylinder length=4.6 radius=0.25
- added link front_axle_mount
- added link front_left_steering_linkage, mass 1.0; visual cylinder length=0.2 radius=0.25
- added link front_right_steering_linkage, mass 1.0; visual cylinder length=0.2 radius=0.25
- added link rear_axle, mass 10.0; visual cylinder length=5.0 radius=0.25
- added link rear_axle_mount
Joints:
- removed joint axle_front_left
- removed joint axle_front_right
- removed joint axle_rear_left
- removed joint axle_rear_right
- removed joint body_to_world
- removed joint floor_to_body
- removed joint grill_to_body
- added joint body_to_floor: type fixed, parent body, child floor, origin xyz=0 0 0.0 rpy=0 0.02 0
- added joint body_to_front_axle_mount: type prismatic, parent body, child front_axle_mount, origin xyz=4.25 0 -1.5 rpy=0 0 0, axis 0 0 1, limit lower=-1.0 upper=0.25
- added joint body_to_grill: type fixed, parent body, child grill, origin xyz=7 0 0
- added joint body_to_rear_axle_mount: type prismatic, parent body, child rear_axle_mount, origin xyz=-3.5 0 -1.5 rpy=0 0 0, axis 0 0 1.0, limit lower=-1.0 upper=0.25
- added joint front_axle_to_left_linkage: type revolute, parent front_axle, child front_left_steering_linkage, origin xyz=0 0 2.3 rpy=0 0 0, axis 0 1 0, limit lower=-0.6 upper=0.6
- added joint front_axle_to_right_linkage: type revolute, parent front_axle, child front_right_steering_linkage, origin xyz=0 0 -2.3 rpy=0 0 0, axis 0 1 0, limit lower=-0.6 upper=0.6
- added joint front_linkage_to_left_wheel: type continuous, parent front_left_steering_linkage, child wheel_front_left, origin xyz=0 0 0.2 rpy=0 0 0, axis 0 0 1
- added joint front_linkage_to_right_wheel: type continuous, parent front_right_steering_linkage, child wheel_front_right, origin xyz=0 0 -0.2 rpy=0 0 0, axis 0 0 1
- added joint mount_to_front_axle: type revolute, parent front_axle_mount, child front_axle, origin xyz=0 0 0 rpy=1.57 0 0, axis 1 0 0, limit lower=-0.4 upper=0.4
- added joint mount_to_rear_axle: type revolute, parent rear_axle_mount, child rear_axle, origin xyz=0 0 0 rpy=1.57 0 0, axis 1 0 0, limit lower=-0.4 upper=0.4
- added joint rear_axle_to_left_wheel: type continuous, parent rear_axle, child wheel_rear_left, origin xyz=0 0 2.5 rpy=0 0 0, axis 0 0 1
- added joint rear_axle_to_right_wheel: type continuous, parent rear_axle, child wheel_rear_right, origin xyz=0 0 -2.5 rpy=0 0 0, axis 0 0 1
- added joint world_to_body: type floating, parent world, child body, origin xyz=0 0 2.6

Commit message: Contact working, adding spring dampers on suspension joints, drop test works

File: src/assets/chevy.urdf (robot description, URDF)
Before this commit: robot Chevy, 13 links, 12 joints
Joints:
- joint body_to_front_axle_mount: limit lower=-1.0 upper=0.25 -> (none); origin xyz=4.25 0 -1.5 rpy=0 0 0 -> xyz=4.25 0 -2.25 rpy=0 0 0
- joint body_to_rear_axle_mount: limit lower=-1.0 upper=0.25 -> (none); origin xyz=-3.5 0 -1.5 rpy=0 0 0 -> xyz=-3.5 0 -2.35 rpy=0 0 0

Commit message: measurements

File: src/assets/chevy.urdf (robot description, URDF)
Before this commit: robot Chevy, 13 links, 12 joints
Links:
- added link camera_1; visual box size=0.4 0.25 0.25
- added link camera_2; visual box size=0.4 0.25 0.25
- added link gps; visual cylinder length=0.5 radius=0.1
- added link imu; visual box size=0.5 0.5 0.2
Joints:
- added joint body_to_camera_1: type fixed, parent body, child camera_1, origin xyz=1.35 1.7 2.4 rpy=0 0.02 0
- added joint body_to_camera_2: type fixed, parent body, child camera_2, origin xyz=1.35 -1.7 2.4 rpy=0 0.02 0
- added joint body_to_gps: type fixed, parent body, child gps, origin xyz=-3.0 1.0 2.6 rpy=0 0 0
- added joint body_to_imu: type fixed, parent body, child imu, origin xyz=0 0 0.7 rpy=0 0.02 0
